Commit message: use .stl files for visualisation

File: ros2srrc_robots/irb14000/urdf/irb14000_macro.urdf.xacro (robot description, xacro)
@@ -83,5 +83,5 @@
         <origin xyz="0 0 0" rpy="0 0 0"/>
         <geometry>
-          <mesh filename="file://$(find ros2srrc_robots)/irb14000/meshes/visual/base_link.dae"/>
+          <mesh filename="file://$(find ros2srrc_robots)/irb14000/meshes/collision/base_link.stl"/>
         </geometry>
         <xacro:material_abb_yellow />
@@ -251,5 +251,5 @@
         <origin xyz="0 0 0" rpy="0 0 0"/>
         <geometry>
-          <mesh filename="file://$(find ros2srrc_robots)/irb14000/meshes/visual/link_1.dae"/>
+          <mesh filename="file://$(find ros2srrc_robots)/irb14000/meshes/collision/link_1.stl"/>
         </geometry>
         <xacro:material_abb_yellow />
@@ -272,5 +272,5 @@
         <origin xyz="0 0 0" rpy="0 0 0"/>
         <geometry>
-          <mesh filename="file://$(find ros2srrc_robots)/irb14000/meshes/visual/link_2.dae"/>
+          <mesh filename="file://$(find ros2srrc_robots)/irb14000/meshes/collision/link_2.stl"/>
         </geometry>
         <xacro:material_abb_yellow />
@@ -293,5 +293,5 @@
         <origin xyz="0 0 0" rpy="0 0 0"/>
         <geometry>
-          <mesh filename="file://$(find ros2srrc_robots)/irb14000/meshes/visual/link_3.dae"/>
+          <mesh filename="file://$(find ros2srrc_robots)/irb14000/meshes/collision/link_3.stl"/>
         </geometry>
         <xacro:material_abb_yellow />
@@ -314,5 +314,5 @@
         <origin xyz="0 0 0" rpy="0 0 0"/>
         <geometry>
-          <mesh filename="file://$(find ros2srrc_robots)/irb14000/meshes/visual/link_4.dae"/>
+          <mesh filename="file://$(find ros2srrc_robots)/irb14000/meshes/collision/link_4.stl"/>
         </geometry>
         <xacro:material_abb_yellow />
@@ -335,5 +335,5 @@
         <origin xyz="0 0 0" rpy="0 0 0"/>
         <geometry>
-          <mesh filename="file://$(find ros2srrc_robots)/irb14000/meshes/visual/link_5.dae"/>
+          <mesh filename="file://$(find ros2srrc_robots)/irb14000/meshes/collision/link_5.stl"/>
         </geometry>
         <xacro:material_abb_yellow />
@@ -356,5 +356,5 @@
         <origin xyz="0 0 0" rpy="0 0 0"/>
         <geometry>
-          <mesh filename="file://$(find ros2srrc_robots)/irb14000/meshes/visual/link_6.dae"/>
+          <mesh filename="file://$(find ros2srrc_robots)/irb14000/meshes/collision/link_6.stl"/>
         </geometry>
         <xacro:material_abb_yellow />
@@ -377,5 +377,5 @@
         <origin xyz="0 0 0" rpy="0 0 0"/>
         <geometry>
-          <mesh filename="file://$(find ros2srrc_robots)/irb14000/meshes/visual/link_7.dae"/>
+          <mesh filename="file://$(find ros2srrc_robots)/irb14000/meshes/collision/link_7.stl"/>
         </geometry>
         <xacro:material_abb_yellow />

Commit message: One arm working in 14000_2

File: ros2srrc_robots/irb14000/urdf/irb14000_macro.urdf.xacro (robot description, xacro)
@@ -67,24 +67,25 @@
     <!-- ***** ABB-IRB1200 ROBOT .urdf SERIAL CHAIN ***** -->
     <!-- Link list: -->
-    <!-- base_link -->
+        <!-- base_link -->
     <link name="base_link">
       <inertial>
-        <mass value="15"/>
-        <origin xyz="0 0 0"/>
-        <inertia ixx="0.5" ixy="0" ixz="0" iyy="0.6" iyz="0" izz="0.3"/>
-      </inertial>
-      <collision name="collision">
-        <origin xyz="0 0 0" rpy="0 0 0"/>
-        <geometry>
-          <mesh filename="file://$(find ros2srrc_robots)/irb14000/meshes/collision/base_link.stl"/>
-        </geometry>
-      </collision>
-      <visual name="visual">
-        <origin xyz="0 0 0" rpy="0 0 0"/>
-        <geometry>
-          <mesh filename="file://$(find ros2srrc_robots)/irb14000/meshes/collision/base_link.stl"/>
-        </geometry>
-        <xacro:material_abb_yellow />
-      </visual>
+        <mass value="6.215"/>
+        <origin xyz="-0.04204 8.01E-05 0.07964" rpy="0 0 0"/>
+        <inertia ixx="0.0247272" ixy="-8.0784E-05" ixz="0.00130902" iyy="0.0491285" iyz="-8.0419E-06" izz="0.0472376"/>
+      </inertial>
+      <visual>
+        <origin xyz="0 0 0" rpy="0 0 0"/>
+        <geometry>
+          <mesh filename="file://$(find ros2srrc_robots)/irb14000_2/meshes/visual/base_link.dae"/>
+        </geometry>
+        <xacro:material_abb_orange />
+      </visual>
+      <collision>
+        <origin xyz="0 0 0" rpy="0 0 0"/>
+        <geometry>
+          <mesh filename="file://$(find ros2srrc_robots)/irb14000_2/meshes/collision/base_link.stl"/>
+        </geometry>
+        <xacro:material_abb_yellow />
+      </collision>
     </link>
     <!-- link_1 -->
@@ -386,5 +387,5 @@
     <!-- joint_1 -->
     <joint type="revolute" name="joint_1_r">
-      <origin xyz="0.05355 -0.0725 0.41492" rpy="-0.9795   -0.5682   -2.3155"/>
+      <origin xyz="0.05355 -0.0725 0.41492" rpy="-0.9795 -0.5682 -2.3155"/>
       <axis xyz="0 0 1"/>
       <parent link="base_link"/>
