Commit message: Two arms working

File: packages/irb14000/ros2srrc_irb14000_gazebo/urdf/irb14000.urdf.xacro (robot description, xacro)
@@ -38,5 +38,5 @@
   <xacro:arg name="EE_name" default="none"/>
   <xacro:property name="EE_name" value="$(arg EE_name)"/>
-  <!-- Include XACRO-MACRO file of the IRB1200: -->
+  <!-- Include XACRO-MACRO file of the IRB120: -->
   <xacro:include filename="$(find ros2srrc_robots)/irb14000/urdf/irb14000_macro.urdf.xacro"/>
   <xacro:irb14000
@@ -51,5 +51,5 @@
       <plugin filename="libgazebo_ros2_control.so" name="gazebo_ros2_control">
         <robot_sim_type>gazebo_ros2_control/GazeboSystem</robot_sim_type>
-        <!-- IRB1200 Controller -->
+        <!-- IRB120 Controller -->
         <parameters>$(find ros2srrc_robots)/irb14000/config/controller.yaml</parameters>
       </plugin>

File: ros2srrc_robots/irb14000/urdf/irb14000_macro.urdf.xacro (robot description, xacro)
@@ -26,5 +26,5 @@
 # ===================================== COPYRIGHT ===================================== #
 #                                                                                       #
-#  Some of the information used to build the ROS2 ABB-IRB1200 .urdf files in this ROS2   #
+#  Some of the information used to build the ROS2 ABB-IRB120 .urdf files in this ROS2   #
 #  repository has been taken from the following resource:                               #
 #       - abb_experimental (https://github.com/ros-industrial/abb_experimental)         #
@@ -50,12 +50,12 @@
   <!-- Include additional ABB-Resources/MATERIALS+COLOUR xacro files: -->
   <xacro:include filename="$(find ros2srrc_robots)/irb14000/urdf/abb_resources/common_materials.xacro"/>
-  <!-- XACRO-MACRO of ABB-IRB1200: -->
+  <!-- XACRO-MACRO of ABB-IRB120: -->
   <xacro:macro name="irb14000" params="bringup robot_ip EE EE_name">
-    <!-- ABB-IRB1200 TRANSMISSION: -->
+    <!-- ABB-IRB120 TRANSMISSION: -->
     <xacro:unless value="${bringup}">
       <xacro:include filename="$(find ros2srrc_robots)/irb14000/urdf/irb14000_transmission.xacro" />
       <xacro:irb14000_transmission />
     </xacro:unless>
-    <!-- ABB-IRB1200 GAZEBO - ROS2_CONTROL: -->
+    <!-- ABB-IRB120 GAZEBO - ROS2_CONTROL: -->
     <xacro:include filename="$(find ros2srrc_robots)/irb14000/urdf/irb14000_ros2control.xacro" />
     <xacro:irb14000_ros2control
@@ -65,7 +65,7 @@
       EE_name="${EE_name}"
     />
-    <!-- ***** ABB-IRB1200 ROBOT .urdf SERIAL CHAIN ***** -->
+    <!-- ***** ABB-IRB120 ROBOT .urdf SERIAL CHAIN ***** -->
     <!-- Link list: -->
-        <!-- base_link -->
+    <!-- base_link -->
     <link name="base_link">
       <inertial>
@@ -77,12 +77,12 @@
         <origin xyz="0 0 0" rpy="0 0 0"/>
         <geometry>
-          <mesh filename="file://$(find ros2srrc_robots)/irb14000_2/meshes/visual/base_link.dae"/>
-        </geometry>
-        <xacro:material_abb_orange />
-      </visual>
-      <collision>
-        <origin xyz="0 0 0" rpy="0 0 0"/>
-        <geometry>
-          <mesh filename="file://$(find ros2srrc_robots)/irb14000_2/meshes/collision/base_link.stl"/>
+          <mesh filename="file://$(find ros2srrc_robots)/irb120/meshes/visual/base_link.dae"/>
+        </geometry>
+        <xacro:material_abb_orange />
+      </visual>
+      <collision>
+        <origin xyz="0 0 0" rpy="0 0 0"/>
+        <geometry>
+          <mesh filename="file://$(find ros2srrc_robots)/irb120/meshes/collision/base_link.stl"/>
         </geometry>
         <xacro:material_abb_yellow />
@@ -90,17 +90,18 @@
     </link>
     <!-- link_1 -->
-    <link name="link_1_r">
-      <inertial>
-        <mass value="1.2"/>
-        <origin xyz="0 -0.03 0.12"/>
-        <inertia ixx="0.1" ixy="0" ixz="0" iyy="0.1" iyz="0" izz="0.1"/>
-      </inertial>
-      <collision name="collision">
+    <link name="link_1">
+      <inertial>
+        <mass value="1.2" />
+        <origin xyz="0 -0.03 0.12" rpy="0 0 0"/>
+        <inertia ixx="0.1" ixy="0" ixz="0" iyy="0.1" iyz="0" izz="0.1"/>
+      </inertial>
+      <visual>
         <origin xyz="0 0 0" rpy="0 0 0"/>
         <geometry>
           <mesh filename="file://$(find ros2srrc_robots)/irb14000/meshes/collision/link_1.stl"/>
         </geometry>
-      </collision>
-      <visual name="visual">
+        <xacro:material_abb_orange />
+      </visual>
+      <collision>
         <origin xyz="0 0 0" rpy="0 0 0"/>
         <geometry>
@@ -108,20 +109,21 @@
         </geometry>
         <xacro:material_abb_yellow />
-      </visual>
+      </collision>
     </link>
     <!-- link_2 -->
-    <link name="link_2_r">
+    <link name="link_2">
       <inertial>
         <mass value="1.6"/>
-        <origin xyz="0 0 0"/>
-         <inertia ixx="0.1" ixy="0" ixz="0" iyy="0.1" iyz="0" izz="0.1"/>
-      </inertial>
-      <collision name="collision">
+        <origin xyz="0 0 0" rpy="0 0 0"/>
+        <inertia ixx="0.1" ixy="0" ixz="0" iyy="0.1" iyz="0" izz="0.1"/>
+      </inertial>
+      <visual>
         <origin xyz="0 0 0" rpy="0 0 0"/>
         <geometry>
           <mesh filename="file://$(find ros2srrc_robots)/irb14000/meshes/collision/link_2.stl"/>
         </geometry>
-      </collision>
-      <visual name="visual">
+        <xacro:material_abb_orange />
+      </visual>
+      <collision>
         <origin xyz="0 0 0" rpy="0 0 0"/>
         <geometry>
@@ -129,20 +131,21 @@
         </geometry>
         <xacro:material_abb_yellow />
-      </visual>
+      </collision>
     </link>
     <!-- link_3 -->
-    <link name="link_3_r">
+    <link name="link_3">
       <inertial>
         <mass value="0.9"/>
-        <origin xyz="0 0 0"/>
-        <inertia ixx="0.1" ixy="0" ixz="0" iyy="0.1" iyz="0" izz="0.1"/>
-      </inertial>
-      <collision name="collision">
+        <origin xyz="0 0 0" rpy="0 0 0"/>
+        <inertia ixx="0.1" ixy="0" ixz="0" iyy="0.1" iyz="0" izz="0.1"/>
+      </inertial>
+      <visual>
         <origin xyz="0 0 0" rpy="0 0 0"/>
         <geometry>
           <mesh filename="file://$(find ros2srrc_robots)/irb14000/meshes/collision/link_3.stl"/>
         </geometry>
-      </collision>
-      <visual name="visual">
+        <xacro:material_abb_orange />
+      </visual>
+      <collision>
         <origin xyz="0 0 0" rpy="0 0 0"/>
         <geometry>
@@ -150,20 +153,21 @@
         </geometry>
         <xacro:material_abb_yellow />
-      </visual>
+      </collision>
     </link>
     <!-- link_4 -->
-    <link name="link_4_r">
+    <link name="link_4">
       <inertial>
         <mass value="1.3"/>
-        <origin xyz="0 0 0"/>
-        <inertia ixx="0.1" ixy="0" ixz="0" iyy="0.1" iyz="0" izz="0.1"/>
-      </inertial>
-      <collision name="collision">
+        <origin xyz="0 0 0" rpy="0 0 0"/>
+        <inertia ixx="0.1" ixy="0" ixz="0" iyy="0.1" iyz="0" izz="0.1"/>
+      </inertial>
+      <visual>
         <origin xyz="0 0 0" rpy="0 0 0"/>
         <geometry>
           <mesh filename="file://$(find ros2srrc_robots)/irb14000/meshes/collision/link_4.stl"/>
         </geometry>
-      </collision>
-      <visual name="visual">
+        <xacro:material_abb_orange />
+      </visual>
+      <collision>
         <origin xyz="0 0 0" rpy="0 0 0"/>
         <geometry>
@@ -171,20 +175,21 @@
         </geometry>
         <xacro:material_abb_yellow />
-      </visual>
+      </collision>
     </link>
     <!-- link_5 -->
-    <link name="link_5_r">
+    <link name="link_5">
       <inertial>
         <mass value="0.5"/>
-        <origin xyz="0 0 0"/>
-         <inertia ixx="0.1" ixy="0" ixz="0" iyy="0.1" iyz="0" izz="0.1"/>
-      </inertial>
-      <collision name="collision">
+        <origin xyz="0 0 0" rpy="0 0 0"/>
+        <inertia ixx="0.1" ixy="0" ixz="0" iyy="0.1" iyz="0" izz="0.1"/>
+      </inertial>
+      <visual>
         <origin xyz="0 0 0" rpy="0 0 0"/>
         <geometry>
           <mesh filename="file://$(find ros2srrc_robots)/irb14000/meshes/collision/link_5.stl"/>
         </geometry>
-      </collision>
-      <visual name="visual">
+        <xacro:material_abb_orange />
+      </visual>
+      <collision>
         <origin xyz="0 0 0" rpy="0 0 0"/>
         <geometry>
@@ -192,20 +197,21 @@
         </geometry>
         <xacro:material_abb_yellow />
-      </visual>
+      </collision>
     </link>
     <!-- link_6 -->
-    <link name="link_6_r">
+    <link name="link_6">
       <inertial>
         <mass value="0.6"/>
-        <origin xyz="0 0 0"/>
-        <inertia ixx="0.1" ixy="0" ixz="0" iyy="0.1" iyz="0" izz="0.1"/>
-      </inertial>
-      <collision name="collision">
+        <origin xyz="0 0 0" rpy="0 0 0"/>
+        <inertia ixx="0.1" ixy="0" ixz="0" iyy="0.1" iyz="0" izz="0.1"/>
+      </inertial>
+      <visual>
         <origin xyz="0 0 0" rpy="0 0 0"/>
         <geometry>
           <mesh filename="file://$(find ros2srrc_robots)/irb14000/meshes/collision/link_6.stl"/>
         </geometry>
-      </collision>
-      <visual name="visual">
+        <xacro:material_abb_black />
+      </visual>
+      <collision>
         <origin xyz="0 0 0" rpy="0 0 0"/>
         <geometry>
@@ -213,20 +219,21 @@
         </geometry>
         <xacro:material_abb_yellow />
-      </visual>
-    </link>
-     <!-- link_7 -->
-    <link name="link_7_r">
+      </collision>
+    </link>
+    <!-- link_7 -->
+    <link name="link_7">
       <inertial>
         <mass value="0.24168"/>
-        <origin xyz="0 0 0"/>
-        <inertia ixx="0.1" ixy="0" ixz="0" iyy="0.1" iyz="0" izz="0.1"/>
-      </inertial>
-      <collision name="collision">
+        <origin xyz="0 0 0" rpy="0 0 0"/>
+        <inertia ixx="0.1" ixy="0" ixz="0" iyy="0.1" iyz="0" izz="0.1"/>
+      </inertial>
+      <visual>
         <origin xyz="0 0 0" rpy="0 0 0"/>
         <geometry>
           <mesh filename="file://$(find ros2srrc_robots)/irb14000/meshes/collision/link_7.stl"/>
         </geometry>
-      </collision>
-      <visual name="visual">
+        <xacro:material_abb_black />
+      </visual>
+      <collision>
         <origin xyz="0 0 0" rpy="0 0 0"/>
         <geometry>
@@ -234,20 +241,21 @@
         </geometry>
         <xacro:material_abb_yellow />
-      </visual>
-    </link>
-        <!-- link_1 -->
-    <link name="link_1_l">
-      <inertial>
-        <mass value="0.9629"/>
-        <origin xyz="0 -0.03 0.12"/>
-        <inertia ixx="0.1" ixy="0" ixz="0" iyy="0.1" iyz="0" izz="0.1"/>
-      </inertial>
-      <collision name="collision">
+      </collision>
+    </link>
+    <!-- link_1 -->
+    <link name="link_8">
+      <inertial>
+        <mass value="1.2" />
+        <origin xyz="0 -0.03 0.12" rpy="0 0 0"/>
+        <inertia ixx="0.1" ixy="0" ixz="0" iyy="0.1" iyz="0" izz="0.1"/>
+      </inertial>
+      <visual>
         <origin xyz="0 0 0" rpy="0 0 0"/>
         <geometry>
           <mesh filename="file://$(find ros2srrc_robots)/irb14000/meshes/collision/link_1.stl"/>
         </geometry>
-      </collision>
-      <visual name="visual">
+        <xacro:material_abb_orange />
+      </visual>
+      <collision>
         <origin xyz="0 0 0" rpy="0 0 0"/>
         <geometry>
@@ -255,20 +263,21 @@
         </geometry>
         <xacro:material_abb_yellow />
-      </visual>
+      </collision>
     </link>
     <!-- link_2 -->
-    <link name="link_2_l">
-      <inertial>
-        <mass value="1.4106"/>
-        <origin xyz="0 0 0"/>
-         <inertia ixx="0.1" ixy="0" ixz="0" iyy="0.1" iyz="0" izz="0.1"/>
-      </inertial>
-      <collision name="collision">
+    <link name="link_9">
+      <inertial>
+        <mass value="1.6"/>
+        <origin xyz="0 0 0" rpy="0 0 0"/>
+        <inertia ixx="0.1" ixy="0" ixz="0" iyy="0.1" iyz="0" izz="0.1"/>
+      </inertial>
+      <visual>
         <origin xyz="0 0 0" rpy="0 0 0"/>
         <geometry>
           <mesh filename="file://$(find ros2srrc_robots)/irb14000/meshes/collision/link_2.stl"/>
         </geometry>
-      </collision>
-      <visual name="visual">
+        <xacro:material_abb_orange />
+      </visual>
+      <collision>
         <origin xyz="0 0 0" rpy="0 0 0"/>
         <geometry>
@@ -276,20 +285,21 @@
         </geometry>
         <xacro:material_abb_yellow />
-      </visual>
+      </collision>
     </link>
     <!-- link_3 -->
-    <link name="link_3_l">
-      <inertial>
-        <mass value="0.7108"/>
-        <origin xyz="0 0 0"/>
-        <inertia ixx="0.1" ixy="0" ixz="0" iyy="0.1" iyz="0" izz="0.1"/>
-      </inertial>
-      <collision name="collision">
+    <link name="link_10">
+      <inertial>
+        <mass value="0.9"/>
+        <origin xyz="0 0 0" rpy="0 0 0"/>
+        <inertia ixx="0.1" ixy="0" ixz="0" iyy="0.1" iyz="0" izz="0.1"/>
+      </inertial>
+      <visual>
         <origin xyz="0 0 0" rpy="0 0 0"/>
         <geometry>
           <mesh filename="file://$(find ros2srrc_robots)/irb14000/meshes/collision/link_3.stl"/>
         </geometry>
-      </collision>
-      <visual name="visual">
+        <xacro:material_abb_orange />
+      </visual>
+      <collision>
         <origin xyz="0 0 0" rpy="0 0 0"/>
         <geometry>
@@ -297,20 +307,21 @@
         </geometry>
         <xacro:material_abb_yellow />
-      </visual>
+      </collision>
     </link>
     <!-- link_4 -->
-    <link name="link_4_l">
-      <inertial>
-        <mass value="1.1808"/>
-        <origin xyz="0 0 0"/>
-        <inertia ixx="0.1" ixy="0" ixz="0" iyy="0.1" iyz="0" izz="0.1"/>
-      </inertial>
-      <collision name="collision">
+    <link name="link_11">
+      <inertial>
+        <mass value="1.3"/>
+        <origin xyz="0 0 0" rpy="0 0 0"/>
+        <inertia ixx="0.1" ixy="0" ixz="0" iyy="0.1" iyz="0" izz="0.1"/>
+      </inertial>
+      <visual>
         <origin xyz="0 0 0" rpy="0 0 0"/>
         <geometry>
           <mesh filename="file://$(find ros2srrc_robots)/irb14000/meshes/collision/link_4.stl"/>
         </geometry>
-      </collision>
-      <visual name="visual">
+        <xacro:material_abb_orange />
+      </visual>
+      <collision>
         <origin xyz="0 0 0" rpy="0 0 0"/>
         <geometry>
@@ -318,20 +329,21 @@
         </geometry>
         <xacro:material_abb_yellow />
-      </visual>
+      </collision>
     </link>
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