Commit message: Two arms working

File: ros2srrc_robots/irb14000/urdf/irb14000_ros2control.xacro (robot description, xacro)
@@ -26,5 +26,5 @@
 # ===================================== COPYRIGHT ===================================== #
 #                                                                                       #
-#  Some of the information used to build the ROS2 ABB-IRB1200 .urdf files in this ROS2   #
+#  Some of the information used to build the ROS2 ABB-IRB120 .urdf files in this ROS2   #
 #  repository has been taken from the following resource:                               #
 #       - abb_experimental (https://github.com/ros-industrial/abb_experimental)         #
@@ -75,13 +75,13 @@
         </hardware>
       </xacro:if>
-      <!-- irb1200_joint1 -->
-      <joint name="joint_1_r">
-        <command_interface name="position">
-          <param name="min">-2.967</param>
-          <param name="max">2.967</param>
-        </command_interface>
-        <command_interface name="velocity">
-          <param name="min">-3.14</param>
-          <param name="max">3.14</param>
+      <!-- irb120_joint1 -->
+      <joint name="joint_1">
+        <command_interface name="position">
+          <param name="min">-2.87979</param>
+          <param name="max">2.87979</param>
+        </command_interface>
+        <command_interface name="velocity">
+          <param name="min">-4.36332</param>
+          <param name="max">4.36332</param>
         </command_interface>
         <state_interface name="position">
@@ -90,12 +90,87 @@
         <state_interface name="velocity"/>
       </joint>
-      <joint name="joint_1_l">
-        <command_interface name="position">
-          <param name="min">-2.967</param>
-          <param name="max">2.967</param>
-        </command_interface>
-        <command_interface name="velocity">
-          <param name="min">-3.14</param>
-          <param name="max">3.14</param>
+      <!-- irb120_joint2 -->
+      <joint name="joint_2">
+        <command_interface name="position">
+          <param name="min">-1.91986</param>
+          <param name="max">1.91986</param>
+        </command_interface>
+        <command_interface name="velocity">
+          <param name="min">-4.36332</param>
+          <param name="max">4.36332</param>
+        </command_interface>
+        <state_interface name="position">
+          <param name="initial_value">-0.785</param>
+        </state_interface>
+        <state_interface name="velocity"/>
+      </joint>
+      <!-- irb120_joint3 -->
+      <joint name="joint_3">
+        <command_interface name="position">
+          <param name="min">-1.91986</param>
+          <param name="max">1.22173</param>
+        </command_interface>
+        <command_interface name="velocity">
+          <param name="min">-4.36332</param>
+          <param name="max">4.36332</param>
+        </command_interface>
+        <state_interface name="position">
+          <param name="initial_value">0.524</param>
+        </state_interface>
+        <state_interface name="velocity"/>
+      </joint>
+      <!-- irb120_joint4 -->
+      <joint name="joint_4">
+        <command_interface name="position">
+          <param name="min">-2.79253</param>
+          <param name="max">2.79253</param>
+        </command_interface>
+        <command_interface name="velocity">
+          <param name="min">-5.58505</param>
+          <param name="max">5.58505</param>
+        </command_interface>
+        <state_interface name="position">
+          <param name="initial_value">-1.309</param>
+        </state_interface>
+        <state_interface name="velocity"/>
+      </joint>
+      <!-- irb120_joint5 -->
+      <joint name="joint_5">
+        <command_interface name="position">
+          <param name="min">-2.00</param>       <!-- Joint5 limits lowered to +-2rad -->
+          <param name="max">2.00</param>
+        </command_interface>
+        <command_interface name="velocity">
+          <param name="min">-5.58505</param>
+          <param name="max">5.58505</param>
+        </command_interface>
+        <state_interface name="position">
+          <param name="initial_value">0.524</param>
+        </state_interface>
+        <state_interface name="velocity"/>
+      </joint>
+      <!-- irb120_joint6 -->
+      <joint name="joint_6">
+        <command_interface name="position">
+          <param name="min">-6.98132</param>
+          <param name="max">6.98132</param>
+        </command_interface>
+        <command_interface name="velocity">
+          <param name="min">-7.33038</param>
+          <param name="max">7.33038</param>
+        </command_interface>
+        <state_interface name="position">
+          <param name="initial_value">-0.349</param>
+        </state_interface>
+        <state_interface name="velocity"/>
+      </joint>
+      <joint name="joint_7">
+        <command_interface name="position">
+          <param name="min">-6.98132</param>
+          <param name="max">6.98132</param>
+        </command_interface>
+        <command_interface name="velocity">
+          <param name="min">-7.33038</param>
+          <param name="max">7.33038</param>
         </command_interface>
         <state_interface name="position">
@@ -104,13 +179,13 @@
         <state_interface name="velocity"/>
       </joint>
-      <!-- irb1200_joint2 -->
-      <joint name="joint_2_r">
-        <command_interface name="position">
-          <param name="min">-2.4</param>
-          <param name="max">0.7</param>
-        </command_interface>
-        <command_interface name="velocity">
-          <param name="min">-3.14</param>
-          <param name="max">3.14</param>
+      <!-- irb120_joint1 -->
+      <joint name="joint_8">
+        <command_interface name="position">
+          <param name="min">-2.87979</param>
+          <param name="max">2.87979</param>
+        </command_interface>
+        <command_interface name="velocity">
+          <param name="min">-4.36332</param>
+          <param name="max">4.36332</param>
         </command_interface>
         <state_interface name="position">
@@ -119,157 +194,87 @@
         <state_interface name="velocity"/>
       </joint>
-       <joint name="joint_2_l">
-        <command_interface name="position">
-          <param name="min">-2.4</param>
-          <param name="max">0.7</param>
-        </command_interface>
-        <command_interface name="velocity">
-          <param name="min">-3.14</param>
-          <param name="max">3.14</param>
-        </command_interface>
-        <state_interface name="position">
-          <param name="initial_value">0.0</param>
+      <!-- irb120_joint2 -->
+      <joint name="joint_9">
+        <command_interface name="position">
+          <param name="min">-1.91986</param>
+          <param name="max">1.91986</param>
+        </command_interface>
+        <command_interface name="velocity">
+          <param name="min">-4.36332</param>
+          <param name="max">4.36332</param>
+        </command_interface>
+        <state_interface name="position">
+          <param name="initial_value">0</param>
         </state_interface>
         <state_interface name="velocity"/>
       </joint>
       <!-- irb120_joint3 -->
-      <joint name="joint_7_r">
-        <command_interface name="position">
-          <param name="min">-2.9</param>
-          <param name="max">2.9</param>
-        </command_interface>
-        <command_interface name="velocity">
-          <param name="min">-3.14</param>
-          <param name="max">3.14</param>
-        </command_interface>
-        <state_interface name="position">
-          <param name="initial_value">0.0</param>
-        </state_interface>
-        <state_interface name="velocity"/>
-      </joint>
-      <joint name="joint_7_l">
-        <command_interface name="position">
-          <param name="min">-2.9</param>
-          <param name="max">2.9</param>
-        </command_interface>
-        <command_interface name="velocity">
-          <param name="min">-3.14</param>
-          <param name="max">3.14</param>
-        </command_interface>
-        <state_interface name="position">
-          <param name="initial_value">0.0</param>
-        </state_interface>
-        <state_interface name="velocity"/>
-      </joint>
-      <!-- irb1200_joint4 -->
-      <joint name="joint_3_r">
-        <command_interface name="position">
-          <param name="min">-2.12</param>
-          <param name="max">1.3</param>
-        </command_interface>
-        <command_interface name="velocity">
-          <param name="min">-3.14</param>
-          <param name="max">3.14</param>
-        </command_interface>
-        <state_interface name="position">
-          <param name="initial_value">0.0</param>
-        </state_interface>
-        <state_interface name="velocity"/>
-      </joint>
-      <joint name="joint_3_l">
-        <command_interface name="position">
-          <param name="min">-2.12</param>
-          <param name="max">1.3</param>
-        </command_interface>
-        <command_interface name="velocity">
-          <param name="min">-3.14</param>
-          <param name="max">3.14</param>
-        </command_interface>
-        <state_interface name="position">
-          <param name="initial_value">0.0</param>
-        </state_interface>
-        <state_interface name="velocity"/>
-      </joint>
-      <!-- irb1200_joint5 -->
-      <joint name="joint_4_r">
-        <command_interface name="position">
-          <param name="min">-5</param>       <!-- Joint5 limits lowered to +-2rad -->
-          <param name="max">5</param>
-        </command_interface>
-        <command_interface name="velocity">
-          <param name="min">-6.98</param>
-          <param name="max">6.98</param>
-        </command_interface>
-        <state_interface name="position">
-          <param name="initial_value">0.0</param>
-        </state_interface>
-        <state_interface name="velocity"/>
-      </joint>
-      <joint name="joint_4_l">
-        <command_interface name="position">
-          <param name="min">-5</param>       <!-- Joint5 limits lowered to +-2rad -->
-          <param name="max">5</param>
-        </command_interface>
-        <command_interface name="velocity">
-          <param name="min">-6.98</param>
-          <param name="max">6.98</param>
-        </command_interface>
-        <state_interface name="position">
-          <param name="initial_value">0.0</param>
-        </state_interface>
-        <state_interface name="velocity"/>
-      </joint>
-      <!-- irb1200_joint6 -->
-      <joint name="joint_6_r">
-        <command_interface name="position">
-          <param name="min">-3.9</param>
-          <param name="max">3.9</param>
-        </command_interface>
-        <command_interface name="velocity">
-          <param name="min">-6.98</param>
-          <param name="max">6.98</param>
-        </command_interface>
-        <state_interface name="position">
-          <param name="initial_value">0.0</param>
-        </state_interface>
-        <state_interface name="velocity"/>
-      </joint>
-       <joint name="joint_6_l">
-        <command_interface name="position">
-          <param name="min">-3.9</param>
-          <param name="max">3.9</param>
-        </command_interface>
-        <command_interface name="velocity">
-          <param name="min">-6.98</param>
-          <param name="max">6.98</param>
-        </command_interface>
-        <state_interface name="position">
-          <param name="initial_value">0.0</param>
-        </state_interface>
-        <state_interface name="velocity"/>
-      </joint>
-      <!-- irb1200_joint7 -->
-      <joint name="joint_5_r">
-        <command_interface name="position">
-          <param name="min">-1.5</param>
-          <param name="max">2.4</param>
-        </command_interface>
-        <command_interface name="velocity">
-          <param name="min">-6.98</param>
-          <param name="max">6.98</param>
-        </command_interface>
-        <state_interface name="position">
-          <param name="initial_value">0.0</param>
-        </state_interface>
-        <state_interface name="velocity"/>
-      </joint>
-       <joint name="joint_5_l">
-        <command_interface name="position">
-          <param name="min">-1.5</param>
-          <param name="max">2.4</param>
-        </command_interface>
-        <command_interface name="velocity">
-          <param name="min">-6.98</param>
-          <param name="max">6.98</param>
+      <joint name="joint_10">
+        <command_interface name="position">
+          <param name="min">-1.91986</param>
+          <param name="max">1.22173</param>
+        </command_interface>
+        <command_interface name="velocity">
+          <param name="min">-4.36332</param>
+          <param name="max">4.36332</param>
+        </command_interface>
+        <state_interface name="position">
+          <param name="initial_value">0</param>
+        </state_interface>
+        <state_interface name="velocity"/>
+      </joint>
+      <!-- irb120_joint4 -->
+      <joint name="joint_11">
+        <command_interface name="position">
+          <param name="min">-2.79253</param>
+          <param name="max">2.79253</param>
+        </command_interface>
+        <command_interface name="velocity">
+          <param name="min">-5.58505</param>
+          <param name="max">5.58505</param>
+        </command_interface>
+        <state_interface name="position">
+          <param name="initial_value">0</param>
+        </state_interface>
+        <state_interface name="velocity"/>
+      </joint>
+      <!-- irb120_joint5 -->
+      <joint name="joint_12">
+        <command_interface name="position">
+          <param name="min">-2.00</param>       <!-- Joint5 limits lowered to +-2rad -->
+          <param name="max">2.00</param>
+        </command_interface>
+        <command_interface name="velocity">
+          <param name="min">-5.58505</param>
+          <param name="max">5.58505</param>
+        </command_interface>
+        <state_interface name="position">
+          <param name="initial_value">0</param>
+        </state_interface>
+        <state_interface name="velocity"/>
+      </joint>
+      <!-- irb120_joint6 -->
+      <joint name="joint_13">
+        <command_interface name="position">
+          <param name="min">-6.98132</param>
+          <param name="max">6.98132</param>
+        </command_interface>
+        <command_interface name="velocity">
+          <param name="min">-7.33038</param>
+          <param name="max">7.33038</param>
+        </command_interface>
+        <state_interface name="position">
+          <param name="initial_value">0</param>
+        </state_interface>
+        <state_interface name="velocity"/>
+      </joint>
+      <joint name="joint_14">
+        <command_interface name="position">
+          <param name="min">-6.98132</param>
+          <param name="max">6.98132</param>
+        </command_interface>
+        <command_interface name="velocity">
+          <param name="min">-7.33038</param>
+          <param name="max">7.33038</param>
         </command_interface>
         <state_interface name="position">
@@ -308,4 +313,31 @@
         <selfCollide>false</selfCollide>
       </gazebo>
+      <gazebo reference="link_7">
+        <selfCollide>false</selfCollide>
+      </gazebo>
+      <gazebo reference="base_link">
+        <selfCollide>false</selfCollide>
+      </gazebo>
+      <gazebo reference="link_8">
+        <selfCollide>false</selfCollide>
+      </gazebo>
+      <gazebo reference="link_9">
+        <selfCollide>false</selfCollide>
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