Commit message: Two arms working

File: ros2srrc_robots/irb14000/urdf/irb14000_transmission.xacro (robot description, xacro)
@@ -26,5 +26,5 @@
 # ===================================== COPYRIGHT ===================================== #
 #                                                                                       #
-#  Some of the information used to build the ROS2 ABB-IRB1200 .urdf files in this ROS2   #
+#  Some of the information used to build the ROS2 ABB-IRB120 .urdf files in this ROS2   #
 #  repository has been taken from the following resource:                               #
 #       - abb_experimental (https://github.com/ros-industrial/abb_experimental)         #
@@ -49,127 +49,127 @@
 <robot xmlns:xacro="http://wiki.ros.org/xacro">
   <xacro:macro name="irb14000_transmission" params="">
-    <transmission name="irb14000_joint1_r_trans">
+    <transmission name="irb14000_joint1_trans">
       <type>transmission_interface/SimpleTransmission</type>
-      <joint name="joint_1_r">
+      <joint name="joint_1">
         <hardwareInterface>hardware_interface/PositionJointInterface</hardwareInterface>
       </joint>
-      <actuator name="irb14000_joint1_r_motor">
+      <actuator name="irb14000_joint1_motor">
         <mechanicalReduction>1</mechanicalReduction>
       </actuator>
     </transmission>
-    <transmission name="irb14000_joint2_r_trans">
+    <transmission name="irb14000_joint2_trans">
       <type>transmission_interface/SimpleTransmission</type>
-      <joint name="joint_2_r">
+      <joint name="joint_2">
         <hardwareInterface>hardware_interface/PositionJointInterface</hardwareInterface>
       </joint>
-      <actuator name="irb14000_joint2_r_motor">
+      <actuator name="irb14000_joint2_motor">
         <mechanicalReduction>1</mechanicalReduction>
       </actuator>
     </transmission>
-    <transmission name="irb14000_joint3_r_trans">
+    <transmission name="irb14000_joint3_trans">
       <type>transmission_interface/SimpleTransmission</type>
-      <joint name="joint_3_r">
+      <joint name="joint_3">
         <hardwareInterface>hardware_interface/PositionJointInterface</hardwareInterface>
       </joint>
-      <actuator name="irb14000_joint3_r_motor">
+      <actuator name="irb14000_joint3_motor">
         <mechanicalReduction>1</mechanicalReduction>
       </actuator>
     </transmission>
-    <transmission name="irb14000_joint4_r_trans">
+    <transmission name="irb14000_joint4_trans">
       <type>transmission_interface/SimpleTransmission</type>
-      <joint name="joint_4_r">
+      <joint name="joint_4">
         <hardwareInterface>hardware_interface/PositionJointInterface</hardwareInterface>
       </joint>
-      <actuator name="irb14000_joint4_r_motor">
+      <actuator name="irb14000_joint4_motor">
         <mechanicalReduction>1</mechanicalReduction>
       </actuator>
     </transmission>
-    <transmission name="irb14000_joint5_r_trans">
+    <transmission name="irb14000_joint5_trans">
       <type>transmission_interface/SimpleTransmission</type>
-      <joint name="joint_5_r">
+      <joint name="joint_5">
         <hardwareInterface>hardware_interface/PositionJointInterface</hardwareInterface>
       </joint>
-      <actuator name="irb14000_joint5_r_motor">
+      <actuator name="irb14000_joint5_motor">
         <mechanicalReduction>1</mechanicalReduction>
       </actuator>
     </transmission>
-    <transmission name="irb14000_joint6_r_trans">
+    <transmission name="irb14000_joint6_trans">
       <type>transmission_interface/SimpleTransmission</type>
-      <joint name="joint_6_r">
+      <joint name="joint_6">
         <hardwareInterface>hardware_interface/PositionJointInterface</hardwareInterface>
       </joint>
-      <actuator name="irb14000_joint6_r_motor">
+      <actuator name="irb14000_joint6_motor">
         <mechanicalReduction>1</mechanicalReduction>
       </actuator>
     </transmission>
-    <transmission name="irb14000_joint7_r_trans">
+    <transmission name="irb14000_joint7_trans">
       <type>transmission_interface/SimpleTransmission</type>
-      <joint name="joint_7_r">
+      <joint name="joint_7">
         <hardwareInterface>hardware_interface/PositionJointInterface</hardwareInterface>
       </joint>
-      <actuator name="irb14000_joint7_r_motor">
+      <actuator name="irb14000_joint7_motor">
         <mechanicalReduction>1</mechanicalReduction>
       </actuator>
     </transmission>
-    <transmission name="irb14000_joint1_l_trans">
+    <transmission name="irb14000_joint8_trans">
       <type>transmission_interface/SimpleTransmission</type>
-      <joint name="joint_1_l">
+      <joint name="joint_8">
         <hardwareInterface>hardware_interface/PositionJointInterface</hardwareInterface>
       </joint>
-      <actuator name="irb14000_joint1_l_motor">
+      <actuator name="irb14000_joint8_motor">
         <mechanicalReduction>1</mechanicalReduction>
       </actuator>
     </transmission>
-    <transmission name="irb14000_joint2_l_trans">
+    <transmission name="irb14000_joint9_trans">
       <type>transmission_interface/SimpleTransmission</type>
-      <joint name="joint_2_l">
+      <joint name="joint_9">
         <hardwareInterface>hardware_interface/PositionJointInterface</hardwareInterface>
       </joint>
-      <actuator name="irb14000_joint2_l_motor">
+      <actuator name="irb14000_joint9_motor">
         <mechanicalReduction>1</mechanicalReduction>
       </actuator>
     </transmission>
-    <transmission name="irb14000_joint3_l_trans">
+    <transmission name="irb14000_joint10_trans">
       <type>transmission_interface/SimpleTransmission</type>
-      <joint name="joint_3_l">
+      <joint name="joint_10">
         <hardwareInterface>hardware_interface/PositionJointInterface</hardwareInterface>
       </joint>
-      <actuator name="irb14000_joint3_l_motor">
+      <actuator name="irb14000_joint10_motor">
         <mechanicalReduction>1</mechanicalReduction>
       </actuator>
     </transmission>
-    <transmission name="irb14000_joint4_l_trans">
+    <transmission name="irb14000_joint11_trans">
       <type>transmission_interface/SimpleTransmission</type>
-      <joint name="joint_4_l">
+      <joint name="joint_11">
         <hardwareInterface>hardware_interface/PositionJointInterface</hardwareInterface>
       </joint>
-      <actuator name="irb14000_joint4_l_motor">
+      <actuator name="irb14000_joint11_motor">
         <mechanicalReduction>1</mechanicalReduction>
       </actuator>
     </transmission>
-    <transmission name="irb14000_joint5_l_trans">
+    <transmission name="irb14000_joint12_trans">
       <type>transmission_interface/SimpleTransmission</type>
-      <joint name="joint_5_l">
+      <joint name="joint_12">
         <hardwareInterface>hardware_interface/PositionJointInterface</hardwareInterface>
       </joint>
-      <actuator name="irb14000_joint5_l_motor">
+      <actuator name="irb14000_joint12_motor">
         <mechanicalReduction>1</mechanicalReduction>
       </actuator>
     </transmission>
-    <transmission name="irb14000_joint6_l_trans">
+    <transmission name="irb14000_joint13_trans">
       <type>transmission_interface/SimpleTransmission</type>
-      <joint name="joint_6_l">
+      <joint name="joint_13">
         <hardwareInterface>hardware_interface/PositionJointInterface</hardwareInterface>
       </joint>
-      <actuator name="irb14000_joint6_l_motor">
+      <actuator name="irb14000_joint13_motor">
         <mechanicalReduction>1</mechanicalReduction>
       </actuator>
     </transmission>
-    <transmission name="irb14000_joint7_l_trans">
+    <transmission name="irb14000_joint14_trans">
       <type>transmission_interface/SimpleTransmission</type>
-      <joint name="joint_7_l">
+      <joint name="joint_14">
         <hardwareInterface>hardware_interface/PositionJointInterface</hardwareInterface>
       </joint>
-      <actuator name="irb14000_joint7_l_motor">
+      <actuator name="irb14000_joint14_motor">
         <mechanicalReduction>1</mechanicalReduction>
       </actuator>
